File: esp32pcb/esp32pcb.kicad_sch (KiCad schematic)
At the start: 1 part, among them U1 ESP32-S3-MINI-1

Commit message: added a few symbols and wiring and astuasdfuas;dlf stuffs when will i be a master *stares off into the dark wistfully*
Parts:
- removed U1: ESP32-S3-MINI-1, RF_Module:ESP32-S2-MINI-1, symbol RF_Module:ESP32-S3-MINI-1
- added C1: C_Polarized_Small, symbol Device:C_Polarized_Small
- added D1: LL4148, Diode_SMD:D_MiniMELF, symbol Diode:LL4148
- added D2, D4: LED, symbol Device:LED
- added D3: LED_RBGA, symbol Device:LED_RBGA
- added F1: Fuse, symbol Device:Fuse
- added H1, H2, H3, H4: Hole_Pad, symbol Mechanical:MountingHole_Pad
- added J1: Conn_01x04, symbol Connector_Generic:Conn_01x04
- added J2: Screw_Terminal_01x03, symbol Connector:Screw_Terminal_01x03
- added J3: Screw_Terminal_01x08, symbol Connector:Screw_Terminal_01x08
- added J4: Screw_Terminal_01x02, symbol Connector:Screw_Terminal_01x02
- added J5: USB_C_Receptacle_USB2.0_16P, symbol Connector:USB_C_Receptacle_USB2.0_16P
- added K1: RT314A05, Relay_THT:Relay_SPDT_Schrack-RT1-16A-FormC_RM5mm, symbol Relay:RT314A05
- added Q1: UMH3N, Package_TO_SOT_SMD:SOT-363_SC-70-6, symbol Transistor_BJT:UMH3N
- added Q2: BC817, Package_TO_SOT_SMD:SOT-23, symbol Transistor_BJT:BC817
- added R1, R2: 5k1, symbol Device:R_Small
- added SW1: SW_SPST, symbol Switch:SW_SPST
- added U1: ESP32-WROOM-32D, RF_Module:ESP32-WROOM-32D, symbol RF_Module:ESP32-WROOM-32D
- added U2: USBLC6-2P6, Package_TO_SOT_SMD:SOT-666, symbol Power_Protection:USBLC6-2P6
- added U3: CP2104, Package_DFN_QFN:QFN-24-1EP_4x4mm_P0.5mm_EP2.6x2.6mm, symbol Interface_USB:CP2104
- added U4: Si7021-A20, Package_DFN_QFN:DFN-6-1EP_3x3mm_P1mm_EP1.5x2.4mm, symbol Sensor_Humidity:Si7021-A20
- added U5: 74HC245, symbol 74xx:74HC245
- added U6: LM1117LD-3.3, Package_SON:WSON-8-1EP_4x4mm_P0.8mm_EP2.2x3mm, symbol Regulator_Linear:LM1117LD-3.3
Connections:
- net GND: now also J5.A1 (GND), J5.A12 (GND), J5.B1 (GND), J5.B12 (GND), J5.S1 (SHIELD), R1.2, R2.2, U2.2 (GND)
- new net: U2.1 (I/O1), U3.4 (D-)
- new net: J5.A7 (D-), J5.B7 (D-), U2.3 (I/O2)
- new net: J5.A6 (D+), J5.B6 (D+), U2.4 (I/O2)
- new net: U2.6 (I/O1), U3.3 (D+)
- new net: U6.2 (VI), U6.3 (VI), U6.4 (VI)
- new net: U6.5 (VO), U6.6 (VO), U6.7 (VO), U6.9 (VO)
- new net: J5.A5 (CC1), R2.1
- new net: U3.2 (GND), U3.25 (GND)
- new net: J5.B5 (CC2), R1.1
- new net: U1.1 (GND), U1.15 (GND), U1.38 (GND), U1.39 (GND)
- new net +5VP: J5.A4 (VBUS), J5.A9 (VBUS), J5.B4 (VBUS), J5.B9 (VBUS)
Other:
- company: (none) -> @shelx
- title: (none) -> esp32_board
