File: esp32pcb/esp32pcb.kicad_sch (KiCad schematic)
At the start: 41 parts, among them J1 Conn_01x04, J2 Screw_Terminal_01x03, J3 Screw_Terminal_01x08, J4 Screw_Terminal_01x02, J5 USB_C_Receptacle_USB2.0_16P, K1 RT314A05, Q1 UMH3N, Q2 BC817, SW1 SW_SPST, U1 ESP32-WROOM-32D, U2 USBLC6-2P6, U3 CP2104, U4 Si7021-A20, U5 74HC245, U6 TLV1117LV-3.3

Commit message: rgb lights!!!!!!!!!1 among other things
Parts:
- added C10, C11, C13, C14, C15, C16: 100n, symbol Device:C_Small
- added C12, C17: 22u, symbol Device:C_Small
- added R10, R8, R9: 1K, symbol Device:R_Small
- added R11, R14, R16, R21, R7: 10k, symbol Device:R_Small
- added R12, R13: 4K7, symbol Device:R_Small
- added R15: 1k, symbol Device:R_Small
- added R17, R18, R19, R20, R22, R23: 22R, symbol Device:R_Small
- C1: value C_Polarized_Small -> 1000u/25V
- D2: value LED -> YELLOW
- U5: value 74HC245 -> 74AHCT245
Connections:
- net +3.3V: now also D3.4 (A), J1.2 (Pin_2), U1.2 (VDD), U4.5 (VDD), C12.1, C13.1, C16.1, C17.1, R11.1, R12.1, R13.1, R21.1, R7.1
- net +5VP: now also D1.1 (K), K1.A1, R16.1
- net EN: now also U1.3 (EN), C15.1, R21.2
- net GND: now also C1.2, H1.1, H2.1, H3.1, H4.1, J1.1 (Pin_1), J3.7 (Pin_7), J3.8 (Pin_8), J4.2 (Pin_2), Q2.2 (E), SW1.1 (A), U4.2 (GND), U4.7 (PAD), U5.10 (GND), U5.19 (CE), U5.6 (A4), U5.7 (A5), U5.8 (A6), U5.9 (A7), C11.2, C12.2, C13.2, C14.2, C15.2, C16.2, C17.2, R14.2
- net RX: now also R22.2
- net TX: now also R23.2
- net at D1.2 (A): now also D2.1 (K), K1.A2, Q2.3 (C)
- net at K1.11: now also J2.2 (Pin_2)
- net at K1.12: now also J2.1 (Pin_1)
- net at K1.14: now also J2.3 (Pin_3)
- net at C1.1: now also F1.1, J4.1 (Pin_1)
- net at Q2.1 (B): now also R14.1, R15.2
- net at J3.1 (Pin_1): now also F1.2, J3.2 (Pin_2)
- net at J3.3 (Pin_3): now also R17.2
- net at J3.4 (Pin_4): now also R18.2
- net at J3.5 (Pin_5): now also R19.2
- net at J3.6 (Pin_6): now also R20.2
- net SDA: now reaches J1.3 (Pin_3)
- net SDA: now also U4.1 (SDA), R12.2
- net SCL: now reaches J1.4 (Pin_4)
- net SCL: now also U4.6 (SCL), R13.2
- net SW: now reaches SW1.2 (B)
- net SW: now also C10.1, C11.1, R11.2, R7.2
- net at D3.1 (RK): now also R8.2
- net at D3.2 (BK): now also R10.2
- net at D3.3 (GK): now also R9.2
- net at D2.2 (A): now also R16.2
- net +5V: now reaches U5.1 (A->B)
- net +5V: now also U5.20 (VCC), C14.1
- net at U5.15 (B3): now also R20.1
- net at U5.16 (B2): now also R19.1
- net at U5.17 (B1): now also R18.1
- net at U5.18 (B0): now also R17.1
- net LEDSTR1: now reaches U5.2 (A0)
- net LEDSTR2: now reaches U5.3 (A1)
- net LEDSTR3: now reaches U5.4 (A2)
- net LEDSTR4: now reaches U5.5 (A3)
- new net LED_B: R10.1
- new net LED_G: R9.1
- new net LED_R: R8.1
- new net RELAY: R15.1
- no-connect marks 0 -> 4
Other:
- note added: "GND"
- note added: "QWIIC"
- note added: "SCL"
- note added: "SDA"
- note added: "VCC"
- moved on the sheet: C1, D1, D2, D3, F1, H1, H2, H3, H4, J1, J2, J3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
